File: display.kicad_sch (KiCad schematic)
At the start: 8 parts, among them J6 52745-2097, U10 TPS61165DRV

Commit message: Minor edits to layout. Added extra models.
Parts:
- added R14: 100k, Resistor_SMD:R_0402_1005Metric, symbol Device:R_US
- renumbered C51 to C65, C53 to C66, C52 to C67, D1 to D4, L2 to L4, R7 to R13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
Connections:
- net BL_PWM: now also R14.1
- net GND: now also R14.2
Other:
- note added: "Display: E50RA-I-MW550-N"
- moved on the sheet: C65, C66, C67, R13
