File: gps.kicad_sch (KiCad schematic)
At the start: 7 parts, among them J1 732512200, U3 NEO-M8U

Commit message: Minor edits to layout. Added extra models.
Parts:
- added C62, C63: 1u, Capacitor_SMD:C_0402_1005Metric, symbol Device:C
- added U10: TPS22917DBV, Package_TO_SOT_SMD:SOT-23-6, symbol Power_Management:TPS22917DBV
- renumbered C40 to C64, FB1 to FB2, J1 to J5, R2 to R10, R3 to R11, R4 to R12, U3 to U9
Connections:
- net +3.3V: now also C62.1, U10.1 (VIN); no longer R10.1, U9.2 (DSEL), U9.23 (VDD), U9.7 (VDD_USB), U9.9 (VCC_RF)
- net GND: now also C62.2, C63.2, U10.2 (GND)
- new net GPS_EN: U10.3 (ON)
- new net GPS_VDD: C63.1, R10.1, U10.5 (QOD), U10.6 (VOUT), U9.2 (DSEL), U9.23 (VDD), U9.7 (VDD_USB), U9.9 (VCC_RF)
- no-connect marks 3 -> 4
Other:
- moved on the sheet: C64, FB2, J5, R10, R11, R12
