File: lux25-display-pcb.kicad_sch (KiCad schematic)
At the start: 0 parts

Commit message: Finished Layout
Parts:
- added C55, C56: 0.1u, Capacitor_SMD:C_0402_1005Metric, symbol Device:C
- added C57, C58: 10u, Capacitor_SMD:C_0603_1608Metric, symbol Device:C
- added C59, C60, C61, C62: 22u, Capacitor_SMD:C_0805_2012Metric, symbol Device:C
- added C63: 1u, Capacitor_SMD:C_0402_1005Metric, symbol Device:C
- added J3: 43045-0200, Molex_Custom:Molex_Micro-Fit_3.0_43045-0200_2x01_P3.00mm_Horizontal, symbol Connector_Generic:Conn_01x02
- added L3: 3.3u, Inductor_SMD:L_Vishay_IHLP-2020, symbol Device:L
- added L4: 4.7u, Inductor_SMD:L_Vishay_IHLP-2020, symbol Device:L
- added NT2: NetTie_2, NetTies:NetTie_2_0.25mm, symbol Device:NetTie_2
- added R10, R11: 22.1k, Resistor_SMD:R_0402_1005Metric, symbol Device:R_US
- added R8: 73.2k, Resistor_SMD:R_0402_1005Metric, symbol Device:R_US
- added R9: 124k, Resistor_SMD:R_0402_1005Metric, symbol Device:R_US
- added U1: TPS542941, Package_DFN_QFN:Texas_RSA_VQFN-16-1EP_4x4mm_P0.65mm_EP2.7x2.7mm_ThermalVias, symbol TexasInstruments:TPS542941RSA
Connections:
- new net: C63.2, U1.11 (VREG5)
- new net: R11.1, R9.2, U1.12 (VFB2)
- new net: C56.2, L4.1, U1.16 (SW2)
- new net: C56.1, U1.1 (VBST2)
- new net: R10.1, R8.2, U1.9 (VFB1)
- new net: C55.1, L3.1, U1.5 (SW1)
- new net: C55.2, U1.4 (VBST1)
- new net +12V: C57.2, C58.2, J3.2 (Pin_2), U1.14 (EN2), U1.2 (VIN2), U1.3 (VIN1), U1.7 (EN1)
- new net +3.3V: C59.2, C60.2, L3.2, R8.1
- new net +5V: C61.2, C62.2, L4.2, R9.1
- new net GND: C57.1, C58.1, C59.1, C60.1, C61.1, C62.1, J3.1 (Pin_1), NT2.2, U1.15 (PGND2), U1.17 (EP), U1.6 (PGND1)
- new net SGND: C63.1, NT2.1, R10.2, R11.2, U1.10 (GND)
Other:
- added sheet Display (display.kicad_sch)
- added sheet GPS (gps.kicad_sch)
- sheet MCU ports: added BL_PWM, DISPLAY_TE, DISPLAY_~{RESET}, DSI_CLKN, DSI_CLKP, DSI_DSI0N, DSI_DSI0P, DSI_DSI1N, DSI_DSI1P, GPS_EXTINT, GPS_RX, GPS_TIMEPULSE, GPS_TX, GPS_~{RESET}, GPS_~{SAFEBOOT}; removed none

Commit message: Minor edits to layout. Added extra models.
Parts:
- J1: renamed from J3; value 43045-0200 -> 43045-0201
- renumbered C55 to C1, C56 to C2, C57 to C3, C58 to C4, C59 to C5, C60 to C6, C61 to C7, C62 to C8, C63 to C9, L3 to L1, L4 to L2, NT2 to NT1, R8 to R1, R9 to R2, R10 to R3, R11 to R4
Other:
- sheet GPS ports: added GPS_EN; removed none
- sheet MCU ports: added GPS_EN; removed none
Changed lines of the file:
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@@
+	(wire
+		(pts
+			(xy 82.55 60.96) (xy 95.25 60.96)
+		)
+		(stroke
+			(width 0)
+			(type default)
+		)
+	)
 	(wire
 		(pts
@@
 		(on_board yes)
 		(dnp no)
-		(property "Reference" "C63"
+		(property "Reference" "C9"
 			(at 88.265 157.48 0)
 			(effects
@@
 			(project "lux25-display-pcb"
 				(path "/4a69e920-c063-4171-ad7b-68c97b0cb851"
-					(reference "C63")
+					(reference "C9")
 					(unit 1)
 				)
@@
 		(on_board yes)
 		(dnp no)
-		(property "Reference" "#PWR065"
+		(property "Reference" "#PWR08"
 			(at 107.315 168.91 0)
 			(effects
@@
 			(project "lux25-display-pcb"
 				(path "/4a69e920-c063-4171-ad7b-68c97b0cb851"
-					(reference "#PWR065")
+					(reference "#PWR08")
 					(unit 1)
 				)
@@
 		(on_board yes)
 		(dnp no)
-		(property "Reference" "R9"
+		(property "Reference" "R2"
 			(at 152.4 146.05 0)
 			(effects
@@
 			(project "lux25-display-pcb"
 				(path "/4a69e920-c063-4171-ad7b-68c97b0cb851"
-					(reference "R9")
+					(reference "R2")
 					(unit 1)
 				)
@@
 		(dnp no)
 		(fields_autoplaced yes)
-		(property "Reference" "#PWR060"
+		(property "Reference" "#PWR01"
 			(at 104.775 129.54 0)
 			(effects
@@
 			(project "lux25-display-pcb"
 				(path "/4a69e920-c063-4171-ad7b-68c97b0cb851"
-					(reference "#PWR060")
+					(reference "#PWR01")
 					(unit 1)
 				)
@@
 		(on_board yes)
 		(dnp no)
-		(property "Reference" "C58"
+		(property "Reference" "C4"
 			(at 125.095 143.51 0)
 			(effects
@@
 			(project "lux25-display-pcb"
 				(path "/4a69e920-c063-4171-ad7b-68c97b0cb851"
-					(reference "C58")
+					(reference "C4")
 					(unit 1)
 				)
@@
 		(on_board yes)
 		(dnp no)
-		(property "Reference" "L4"
+		(property "Reference" "L2"
 			(at 133.35 137.16 90)
 			(effects
@@
 			(project "lux25-display-pcb"
 				(path "/4a69e920-c063-4171-ad7b-68c97b0cb851"
-					(reference "L4")
+					(reference "L2")
 					(unit 1)
 				)
@@
 		(on_board yes)
 		(dnp no)
-		(property "Reference" "C56"
+		(property "Reference" "C2"
 			(at 121.92 133.985 90)
 			(effects
@@
 			(project "lux25-display-pcb"
 				(path "/4a69e920-c063-4171-ad7b-68c97b0cb851"
-					(reference "C56")
+					(reference "C2")
 					(unit 1)
 				)
@@
 		(on_board yes)
 		(dnp no)
-		(property "Reference" "C61"
+		(property "Reference" "C7"
 			(at 137.795 143.51 0)
 			(effects
@@
 			(project "lux25-display-pcb"
 				(path "/4a69e920-c063-4171-ad7b-68c97b0cb851"
-					(reference "C61")
+					(reference "C7")
 					(unit 1)
 				)
@@
 		(on_board yes)
 		(dnp no)
-		(property "Reference" "#PWR064"
+		(property "Reference" "#PWR06"
 			(at 138.43 156.21 0)
 			(effects
@@
 			(project "lux25-display-pcb"
 				(path "/4a69e920-c063-4171-ad7b-68c97b0cb851"
-					(reference "#PWR064")
+					(reference "#PWR06")
 					(unit 1)
 				)
@@
 		(on_board yes)
 		(dnp no)
-		(property "Reference" "R10"
+		(property "Reference" "R3"
 			(at 59.055 156.21 0)
 			(effects
@@
 			(project "lux25-display-pcb"
 				(path "/4a69e920-c063-4171-ad7b-68c97b0cb851"
-					(reference "R10")
+					(reference "R3")
 					(unit 1)
 				)
@@
 		(on_board yes)
 		(dnp no)
-		(property "Reference" "C57"
+		(property "Reference" "C3"
 			(at 84.455 143.51 0)
 			(effects
@@
 			(project "lux25-display-pcb"
 				(path "/4a69e920-c063-4171-ad7b-68c97b0cb851"
-					(reference "C57")
+					(reference "C3")
 					(unit 1)
 				)
@@
 		(on_board yes)
 		(dnp no)
-		(property "Reference" "C60"
+		(property "Reference" "C6"
 			(at 71.755 143.51 0)
 			(effects
@@
 			(project "lux25-display-pcb"
 				(path "/4a69e920-c063-4171-ad7b-68c97b0cb851"
-					(reference "C60")
+					(reference "C6")
 					(unit 1)
 				)
@@
 		(on_board yes)
 		(dnp no)
-		(property "Reference" "R8"
+		(property "Reference" "R1"
 			(at 59.055 146.05 0)
 			(effects
@@
 			(project "lux25-display-pcb"
 				(path "/4a69e920-c063-4171-ad7b-68c97b0cb851"
-					(reference "R8")
+					(reference "R1")
 					(unit 1)
 				)
@@
 		(on_board yes)
 		(dnp no)
-		(property "Reference" "R11"
+		(property "Reference" "R4"
 			(at 152.4 156.21 0)
 			(effects
@@
 			(project "lux25-display-pcb"
 				(path "/4a69e920-c063-4171-ad7b-68c97b0cb851"
-					(reference "R11")
+					(reference "R4")
 					(unit 1)
 				)
@@
 		(on_board yes)
 		(dnp no)
-		(property "Reference" "#PWR063"
+		(property "Reference" "#PWR05"
 			(at 71.12 156.21 0)
 			(effects
@@
 			(project "lux25-display-pcb"
 				(path "/4a69e920-c063-4171-ad7b-68c97b0cb851"
-					(reference "#PWR063")
+					(reference "#PWR05")
 					(unit 1)
 				)
@@
 		(dnp no)
 		(fields_autoplaced yes)
-		(property "Reference" "NT2"
+		(property "Reference" "NT1"
 			(at 104.775 157.48 0)
 			(effects
@@
 			(project "lux25-display-pcb"
 				(path "/4a69e920-c063-4171-ad7b-68c97b0cb851"
-					(reference "NT2")
+					(reference "NT1")
 					(unit 1)
 				)
@@
 		(dnp no)
 		(fields_autoplaced yes)
-		(property "Reference" "#PWR031"
+		(property "Reference" "#PWR04"
 			(at 43.18 152.4 0)
 			(effects
@@
 			(project ""
 				(path "/4a69e920-c063-4171-ad7b-68c97b0cb851"
-					(reference "#PWR031")
+					(reference "#PWR04")
 					(unit 1)
 				)
@@
 		(on_board yes)
 		(dnp no)
-		(property "Reference" "L3"
+		(property "Reference" "L1"
 			(at 76.2 137.16 90)
 			(effects
@@
 			(project "lux25-display-pcb"
 				(path "/4a69e920-c063-4171-ad7b-68c97b0cb851"
-					(reference "L3")
+					(reference "L1")
 					(unit 1)
 				)
@@
 		(on_board yes)
 		(dnp no)
-		(property "Reference" "#PWR062"
+		(property "Reference" "#PWR03"
 			(at 149.86 146.05 0)
 			(effects
@@
 			(project "lux25-display-pcb"
 				(path "/4a69e920-c063-4171-ad7b-68c97b0cb851"
-					(reference "#PWR062")
+					(reference "#PWR03")
 					(unit 1)
 				)
@@
 		(on_board yes)
 		(dnp no)
-		(property "Reference" "#PWR061"
+		(property "Reference" "#PWR02"
 			(at 61.595 146.05 0)
 			(effects
@@
 			(project "lux25-display-pcb"
 				(path "/4a69e920-c063-4171-ad7b-68c97b0cb851"
-					(reference "#PWR061")
+					(reference "#PWR02")
 					(unit 1)
 				)
@@
 		(on_board yes)
 		(dnp no)
-		(property "Reference" "J3"
+		(property "Reference" "J1"
 			(at 34.29 157.48 0)
 			(effects
@@
 			)
 		)
-		(property "Value" "43045-0200"
+		(property "Value" "43045-0201"
 			(at 34.29 154.94 0)
 			(effects
@@
 			(project ""
 				(path "/4a69e920-c063-4171-ad7b-68c97b0cb851"
-					(reference "J3")
+					(reference "J1")
 					(unit 1)
 				)
@@
 		(on_board yes)
 		(dnp no)
-		(property "Reference" "C59"
+		(property "Reference" "C5"
 			(at 70.485 143.51 0)
 			(effects
@@
 			(project "lux25-display-pcb"
 				(path "/4a69e920-c063-4171-ad7b-68c97b0cb851"
-					(reference "C59")
+					(reference "C5")
 					(unit 1)
 				)
@@
 		(on_board yes)
 		(dnp no)
-		(property "Reference" "C55"
+		(property "Reference" "C1"
 			(at 87.63 133.985 90)
 			(effects
@@
 			(project "lux25-display-pcb"
 				(path "/4a69e920-c063-4171-ad7b-68c97b0cb851"
-					(reference "C55")
+					(reference "C1")
 					(unit 1)
 				)
@@
 		(on_board yes)
 		(dnp no)
-		(property "Reference" "C62"
+		(property "Reference" "C8"
 			(at 139.065 143.51 0)
 			(effects
@@
 			(project "lux25-display-pcb"
 				(path "/4a69e920-c063-4171-ad7b-68c97b0cb851"
-					(reference "C62")
+					(reference "C8")
 					(unit 1)
 				)
@@
 		(dnp no)
 		(fields_autoplaced yes)
-		(property "Reference" "#PWR032"
+		(property "Reference" "#PWR07"
 			(at 43.18 157.48 0)
 			(effects
@@
 			(project ""
 				(path "/4a69e920-c063-4171-ad7b-68c97b0cb851"
-					(reference "#PWR032")
+					(reference "#PWR07")
 					(unit 1)
 				)
@@
 			)
 		)
+		(pin "GPS_EN" input
+			(at 95.25 60.96 180)
+			(effects
+				(font
+					(size 1.27 1.27)
+				)
+				(justify left)
+			)
+		)
 		(instances
 			(project "lux25-display-pcb"
@@
 			(effects
 				(font
+					(size 1.27 1.27)
+				)
+				(justify right)
+			)
+		)
+		(pin "GPS_EN" output
+			(at 82.55 60.96 0)
+			(effects
+				(font
